File: PCB/schematics-v02/kicad/hamodule.kicad_sch (KiCad schematic)
At the start: 9 parts, among them J1 Conn_01x05_Female, J2 Conn_01x05_Female

Commit message: V2 iteration 1
Parts:
- gave numbers to parts that had none: 2
Changed lines of the file:
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@@
   (symbol (lib_id "Connector:TestPoint_2Pole") (at 44.45 54.61 0) (unit 1)
     (in_bom yes) (on_board yes)
-    (property "Reference" "TP?" (id 0) (at 44.45 57.15 0))
+    (property "Reference" "TP2" (id 0) (at 44.45 57.15 0))
     (property "Value" "TestPoint_2Pole" (id 1) (at 44.45 59.69 0))
     (property "Footprint" "" (id 2) (at 44.45 54.61 0)
@@
   (symbol (lib_id "Connector:TestPoint_2Pole") (at 44.45 43.18 0) (unit 1)
     (in_bom yes) (on_board yes) (fields_autoplaced)
-    (property "Reference" "TP?" (id 0) (at 44.45 36.83 0))
+    (property "Reference" "TP1" (id 0) (at 44.45 36.83 0))
     (property "Value" "TestPoint_2Pole" (id 1) (at 44.45 39.37 0))
     (property "Footprint" "" (id 2) (at 44.45 43.18 0)
@@
       (reference "J2") (unit 1) (value "Conn_01x05_Female") (footprint "Connector_PinSocket_2.54mm:PinSocket_1x05_P2.54mm_Vertical")
     )
+    (path "/b9703584-d14d-4010-8f01-295e52d82c0f"
+      (reference "TP1") (unit 1) (value "TestPoint_2Pole") (footprint "")
+    )
     (path "/921f3709-2de6-4205-a9b4-54d0fdceb3f6"
-      (reference "TP?") (unit 1) (value "TestPoint_2Pole") (footprint "")
-    )
-    (path "/b9703584-d14d-4010-8f01-295e52d82c0f"
-      (reference "TP?") (unit 1) (value "TestPoint_2Pole") (footprint "")
+      (reference "TP2") (unit 1) (value "TestPoint_2Pole") (footprint "")
     )
   )
