File: other-projects/workbench/es32-kicad/workbench/workbench.kicad_pcb (KiCad board)
At the start: 2 copper layers, 56 parts, among them J1 GND|5V, J2 Conn_01x08_Socket, J3 Conn_01x16_Socket, J4 Conn_01x08_Socket, J5 GND|3.3V, J6 Current Jumper, J7 Conn_01x02_Male, J8 USB_C_Receptacle_USB2.0, Q1 SS8050, Q2 SS8050, SW1 USB | PS, SW4 Switch, SW5 Switch, U1 LD1117AV33, U2 74HC595, U3 ULN2803A, U5 CP2102N-A01-GQFN28, U6 MCP23017_SP, U7 74HC595, U8 ESP32-WROOM-32D, U9 ULN2803A

Commit message: workbench PCB update
Parts:
- removed C1, C10, C13, C5, C8: 100nF, Capacitor_SMD:C_0603_1608Metric_Pad1.08x0.95mm_HandSolder
- removed C11: 4.7uF, Capacitor_SMD:C_0603_1608Metric_Pad1.08x0.95mm_HandSolder
- removed C12: 22uF, Capacitor_SMD:C_0603_1608Metric_Pad1.08x0.95mm_HandSolder
- removed C2, C3, C6, C7: NC, Capacitor_SMD:C_0805_2012Metric_Pad1.18x1.45mm_HandSolder
- removed C4: 10uF, Capacitor_THT:CP_Radial_D6.3mm_P2.50mm
- removed C9: NC, Capacitor_SMD:C_0603_1608Metric_Pad1.08x0.95mm_HandSolder
- removed D1: LED, LED_SMD:LED_0805_2012Metric_Pad1.15x1.40mm_HandSolder
- removed D3, D4, D5: D_TVS, Diode_SMD:D_SOD-523
- removed D6: BAT60A-7, Diode_SMD:D_SOD-323
- removed F1: 250V500mA, Fuse:Fuseholder_TR5_Littelfuse_No560_No460
- removed J1: GND|5V, Connector_JST:JST_XH_B2B-XH-A_1x02_P2.50mm_Vertical
- removed J5: GND|3.3V, Connector_JST:JST_XH_B2B-XH-A_1x02_P2.50mm_Vertical
- removed J6: Current Jumper, Connector_PinHeader_2.54mm:PinHeader_1x02_P2.54mm_Vertical
- removed J7: Conn_01x02_Male, Connector_PinHeader_2.54mm:PinHeader_1x02_P2.54mm_Vertical
- removed J8: USB_C_Receptacle_USB2.0, Connector_USB:USB_C_Receptacle_HRO_TYPE-C-31-M-12
- removed Q1, Q2: SS8050, Package_TO_SOT_SMD:SOT-23
- removed R17: 100Ω, Resistor_SMD:R_0805_2012Metric_Pad1.20x1.40mm_HandSolder
- removed R18, R33, R34: 10kΩ, Resistor_SMD:R_0603_1608Metric_Pad0.98x0.95mm_HandSolder
- removed R23: 150kΩ1w, Resistor_SMD:R_2512_6332Metric_Pad1.40x3.35mm_HandSolder
- removed R24: 22.1kΩ, Resistor_SMD:R_0603_1608Metric_Pad0.98x0.95mm_HandSolder
- removed R25: 47.5kΩ, Resistor_SMD:R_0603_1608Metric_Pad0.98x0.95mm_HandSolder
- removed R26, R27: 5.1kΩ, Resistor_SMD:R_0603_1608Metric_Pad0.98x0.95mm_HandSolder
- removed R28, R32: 1kΩ, Resistor_SMD:R_0603_1608Metric_Pad0.98x0.95mm_HandSolder
- removed R29, R30: 0Ω, Resistor_SMD:R_0805_2012Metric_Pad1.20x1.40mm_HandSolder
- removed R31: 1kΩ, Resistor_SMD:R_1206_3216Metric_Pad1.30x1.75mm_HandSolder
- removed SW1: USB | PS, Connector_PinHeader_2.54mm:PinHeader_1x03_P2.54mm_Vertical
- removed SW4, SW5: Switch, Button_Switch_SMD:SW_SPST_SKQG_WithStem
- removed U1: LD1117AV33, Package_TO_SOT_THT:TO-220-3_Vertical
- removed U5: CP2102N-A01-GQFN28, Package_DFN_QFN:QFN-28-1EP_5x5mm_P0.5mm_EP3.35x3.35mm
- removed U8: ESP32-WROOM-32D, RF_Module:ESP32-WROOM-32D
- added C14: 10uF, Capacitor_THT:CP_Radial_D6.3mm_P2.50mm, F.Cu at (131.1, 72.8)
- added C15: 10uF, Capacitor_THT:CP_Radial_D6.3mm_P2.50mm, F.Cu at (164.5, 93.1)
- added C16: 10uF, Capacitor_THT:CP_Radial_D6.3mm_P2.50mm, F.Cu at (163.8, 116.6)
- added C17: 10uF, Capacitor_THT:CP_Radial_D6.3mm_P2.50mm, F.Cu at (164.6, 69.7)
- added J10: Rotary Encoder, Connector_JST:JST_EH_B4B-EH-A_1x04_P2.50mm_Vertical, F.Cu at (108.5, 8.64)
- added J11: Conn_01x08_Socket, Connector_PinSocket_2.54mm:PinSocket_1x08_P2.54mm_Vertical, F.Cu at (94.3, 82.6)
- added J9: Conn_01x08_Socket, Connector_PinSocket_2.54mm:PinSocket_1x08_P2.54mm_Vertical, F.Cu at (194.4, 99.4)
- added Q3: IRL520, Package_TO_SOT_THT:TO-220-3_Vertical, F.Cu at (165.5, 6.22)
- added R1: R, Resistor_THT:R_Axial_DIN0207_L6.3mm_D2.5mm_P7.62mm_Horizontal, F.Cu at (105.0, 80.3)
- added R10: R, Resistor_THT:R_Axial_DIN0207_L6.3mm_D2.5mm_P7.62mm_Horizontal, F.Cu at (105.0, 73.5)
- added R11: R, Resistor_THT:R_Axial_DIN0207_L6.3mm_D2.5mm_P7.62mm_Horizontal, F.Cu at (105.0, 70.5)
- added R12: R, Resistor_THT:R_Axial_DIN0207_L6.3mm_D2.5mm_P7.62mm_Horizontal, F.Cu at (105.0, 67.4)
- added R13: R, Resistor_THT:R_Axial_DIN0207_L6.3mm_D2.5mm_P7.62mm_Horizontal, F.Cu at (105.0, 64.4)
- added R14: R, Resistor_THT:R_Axial_DIN0207_L6.3mm_D2.5mm_P7.62mm_Horizontal, F.Cu at (105.0, 61.3)
- added R15: R, Resistor_THT:R_Axial_DIN0207_L6.3mm_D2.5mm_P7.62mm_Horizontal, F.Cu at (105.0, 58.3)
- added R16: R, Resistor_THT:R_Axial_DIN0207_L6.3mm_D2.5mm_P7.62mm_Horizontal, F.Cu at (105.0, 55.2)
- added R2: R, Resistor_THT:R_Axial_DIN0207_L6.3mm_D2.5mm_P7.62mm_Horizontal, F.Cu at (105.0, 83.3)
- added R21: 10k, Resistor_THT:R_Axial_DIN0207_L6.3mm_D2.5mm_P7.62mm_Horizontal, F.Cu at (122.0, 2.79)
- added R22: 10k, Resistor_THT:R_Axial_DIN0207_L6.3mm_D2.5mm_P7.62mm_Horizontal, F.Cu at (122.0, 5.84)
- added R3: R, Resistor_THT:R_Axial_DIN0207_L6.3mm_D2.5mm_P7.62mm_Horizontal, F.Cu at (105.0, 86.4)
- added R35: 10k, Resistor_THT:R_Axial_DIN0207_L6.3mm_D2.5mm_P7.62mm_Horizontal, F.Cu at (122.0, 8.89)
- added R4: R, Resistor_THT:R_Axial_DIN0207_L6.3mm_D2.5mm_P7.62mm_Horizontal, F.Cu at (105.0, 89.4)
- added R5: R, Resistor_THT:R_Axial_DIN0207_L6.3mm_D2.5mm_P7.62mm_Horizontal, F.Cu at (105.0, 92.5)
- added R52: 10k, Resistor_THT:R_Axial_DIN0207_L6.3mm_D2.5mm_P7.62mm_Horizontal, F.Cu at (169.9, 3.68)
- added R53: 10k, Resistor_THT:R_Axial_DIN0207_L6.3mm_D2.5mm_P7.62mm_Horizontal, F.Cu at (177.5, 6.73)
- added R6: R, Resistor_THT:R_Axial_DIN0207_L6.3mm_D2.5mm_P7.62mm_Horizontal, F.Cu at (105.0, 95.5)
- added R7: R, Resistor_THT:R_Axial_DIN0207_L6.3mm_D2.5mm_P7.62mm_Horizontal, F.Cu at (105.0, 98.6)
- added R8: R, Resistor_THT:R_Axial_DIN0207_L6.3mm_D2.5mm_P7.62mm_Horizontal, F.Cu at (105.0, 101.6)
- added R9: R, Resistor_THT:R_Axial_DIN0207_L6.3mm_D2.5mm_P7.62mm_Horizontal, F.Cu at (105.0, 76.6)
- added RN1: R_Network08, Resistor_THT:R_Array_SIP9, F.Cu at (109.2, 77.5)
- added RN2: R_Network08, Resistor_THT:R_Array_SIP9, F.Cu at (109.2, 80.9)
- added U10: ULN2803A, Package_DIP:DIP-18_W7.62mm_LongPads, F.Cu at (183.1, 99.4)
- added U11: ESP32-DevKitC, Esp:ESP32-DevKitC, F.Cu at (130.9, -5.84)
- added U4: 74HC595, Package_DIP:DIP-16_W7.62mm_Socket_LongPads, F.Cu at (177.0, 117.3)
- J3: value Conn_01x16_Socket -> Conn_01x08_Socket; footprint Connector_PinSocket_2.54mm:PinSocket_1x16_P2.54mm_Vertical -> Connector_PinSocket_2.54mm:PinSocket_1x08_P2.54mm_Vertical
- R19, R20: footprint Resistor_SMD:R_0603_1608Metric_Pad0.98x0.95mm_HandSolder -> Resistor_THT:R_Axial_DIN0207_L6.3mm_D2.5mm_P7.62mm_Horizontal
- moved R20 119.9 mm to (120.3, 20.6)
- moved R19 119.8 mm to (120.3, 17.4)
- moved J3 74.6 mm to (94.0, 75.5), turned to 180 degrees
- moved U3 69.7 mm to (183.3, 51.7)
- moved U2 68.8 mm to (177.4, 69.7)
- moved U9 42.1 mm to (183.3, 75.4)
- moved U7 41.5 mm to (177.3, 93.2)
- moved J2 27.2 mm to (194.6, 75.4)
- moved J4 20.4 mm to (194.6, 51.4)
- moved U6 13.9 mm to (124.5, 93.2), turned to 180 degrees
Connections:
- U2 pad 1: /2 -> /Chan2
- U2 pad 10: unconnected-(U2-~{SRCLR}-Pad10) -> +3.3V
- U2 pad 15: /1 -> /Chan1
- U2 pad 2: /3 -> /Chan3
- U2 pad 3: /4 -> /Chan4
- U2 pad 4: /5 -> /Chan5
- U2 pad 5: /6 -> /Chan6
- U2 pad 6: /7 -> /Chan7
- U2 pad 7: /8 -> /Chan8
- U3 pad 1: /8 -> /Chan8
- U3 pad 2: /7 -> /Chan7
- U3 pad 3: /6 -> /Chan6
- U3 pad 4: /5 -> /Chan5
- U3 pad 5: /4 -> /Chan4
- U3 pad 6: /3 -> /Chan3
- U3 pad 7: /2 -> /Chan2
- U3 pad 8: /1 -> /Chan1
- U7 pad 1: /2 -> /Chan10
- U7 pad 10: unconnected-(U7-~{SRCLR}-Pad10) -> +3.3V
- U7 pad 15: /1 -> /Chan9
- U7 pad 2: /3 -> /Chan11
- U7 pad 3: /4 -> /Chan12
- U7 pad 4: /5 -> /Chan13
- U7 pad 5: /6 -> /Chan14
- U7 pad 6: /7 -> /Chan15
- U7 pad 7: /8 -> /Chan16
- U7 pad 9: unconnected-(U7-QH'-Pad9) -> Net-(U4-SER)
- U9 pad 1: /8 -> /Chan16
- U9 pad 2: /7 -> /Chan15
- U9 pad 3: /6 -> /Chan14
- U9 pad 4: /5 -> /Chan13
- U9 pad 5: /4 -> /Chan12
- U9 pad 6: /3 -> /Chan11
- U9 pad 7: /2 -> /Chan10
- U9 pad 8: /1 -> /Chan9
Routing:
- net Net-(U11-GPIO22): track 0.00 -> 118.8 mm, vias 0 -> 2
- net Net-(U11-GPIO21): track 0.00 -> 113.9 mm, vias 0 -> 2
- net Net-(Q3-D): track 0.00 -> 113.8 mm, vias 0 -> 1
- net Net-(U11-GPIO19): track 0.00 -> 58.3 mm
- net Net-(U11-DAC_2/ADC2_CH9/GPIO26): track 0.00 -> 50.0 mm
- net Net-(U11-ADC2_CH7/GPIO27): track 0.00 -> 49.6 mm
- net Net-(U4-SER): track 0.00 -> 45.4 mm, vias 0 -> 1
- net Net-(RN2-R1): track 0.00 -> 43.2 mm
- net Net-(U2-QH'): track 0.00 -> 41.5 mm, vias 0 -> 1
- net Net-(RN2-R2): track 0.00 -> 39.1 mm
- net Net-(RN2-R3): track 0.00 -> 36.6 mm
- net Net-(RN2-R4): track 0.00 -> 33.7 mm
- net Net-(RN2-R5): track 0.00 -> 29.9 mm
- net Net-(RN1-R8): track 0.00 -> 28.3 mm
- net Net-(RN1-R2): track 0.00 -> 27.2 mm
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- added copper zone on In1.Cu, net +3.3V
- added copper zone on In2.Cu, net GND
Other:
- copper layers 2 -> 4
