File: other-projects/workbench/es32-kicad/workbench/workbench.kicad_sch (KiCad schematic)
At the start: 72 parts, among them J1 GND|5V, J2 Conn_01x08_Socket, J3 Conn_01x16_Socket, J4 Conn_01x08_Socket, J5 GND|3.3V, J6 Current Jumper, J7 Conn_01x02_Male, J8 USB_C_Receptacle_USB2.0, Q1 SS8050, Q2 SS8050, SW1 USB | PS, SW4 Switch, SW5 Switch, U1 LD1117AV33, U2 74HC595, U3 ULN2803A, U5 CP2102N-A01-GQFN28, U6 MCP23017_SP, U7 74HC595, U8 ESP32-WROOM-32D, U9 ULN2803A

Commit message: workbench PCB update
Parts:
- removed C1, C10, C13, C5, C8: 100nF, Capacitor_SMD:C_0603_1608Metric_Pad1.08x0.95mm_HandSolder, symbol Device:C_Polarized_Small
- removed C11: 4.7uF, Capacitor_SMD:C_0603_1608Metric_Pad1.08x0.95mm_HandSolder, symbol Device:C_Polarized_Small
- removed C12: 22uF, Capacitor_SMD:C_0603_1608Metric_Pad1.08x0.95mm_HandSolder, symbol Device:C_Polarized_Small
- removed C2, C3, C6, C7: NC, Capacitor_SMD:C_0805_2012Metric_Pad1.18x1.45mm_HandSolder, symbol Device:C_Polarized_Small
- removed C4: 10uF, Capacitor_THT:CP_Radial_D6.3mm_P2.50mm, symbol Device:C_Polarized_Small
- removed C9: NC, Capacitor_SMD:C_0603_1608Metric_Pad1.08x0.95mm_HandSolder, symbol Device:C_Polarized_Small
- removed D1: LED, LED_SMD:LED_0805_2012Metric_Pad1.15x1.40mm_HandSolder, symbol Device:LED
- removed D3, D4, D5: D_TVS, Diode_SMD:D_SOD-523, symbol Device:D_TVS
- removed D6: BAT60A-7, Diode_SMD:D_SOD-323, symbol Diode:BAT60A
- removed F1: 250V500mA, Fuse:Fuseholder_TR5_Littelfuse_No560_No460, symbol Device:Fuse
- removed J1: GND|5V, Connector_JST:JST_XH_B2B-XH-A_1x02_P2.50mm_Vertical, symbol Connector_Generic:Conn_01x02
- removed J3: Conn_01x16_Socket, Connector_PinSocket_2.54mm:PinSocket_1x16_P2.54mm_Vertical, symbol Connector:Conn_01x16_Socket
- removed J5: GND|3.3V, Connector_JST:JST_XH_B2B-XH-A_1x02_P2.50mm_Vertical, symbol Connector_Generic:Conn_01x02
- removed J6: Current Jumper, Connector_PinHeader_2.54mm:PinHeader_1x02_P2.54mm_Vertical, symbol Jumper:Jumper_2_Bridged
- removed J7: Conn_01x02_Male, Connector_PinHeader_2.54mm:PinHeader_1x02_P2.54mm_Vertical, symbol Connector:Conn_01x02_Male
- removed J8: USB_C_Receptacle_USB2.0, Connector_USB:USB_C_Receptacle_HRO_TYPE-C-31-M-12, symbol Connector:USB_C_Receptacle_USB2.0
- removed Q1, Q2: SS8050, Package_TO_SOT_SMD:SOT-23, symbol Device:Q_NPN_BEC
- removed R17: 100Ω, Resistor_SMD:R_0805_2012Metric_Pad1.20x1.40mm_HandSolder, symbol Device:R
- removed R18, R33, R34: 10kΩ, Resistor_SMD:R_0603_1608Metric_Pad0.98x0.95mm_HandSolder, symbol Device:R
- removed R23: 150kΩ1w, Resistor_SMD:R_2512_6332Metric_Pad1.40x3.35mm_HandSolder, symbol Device:R
- removed R24: 22.1kΩ, Resistor_SMD:R_0603_1608Metric_Pad0.98x0.95mm_HandSolder, symbol Device:R
- removed R25: 47.5kΩ, Resistor_SMD:R_0603_1608Metric_Pad0.98x0.95mm_HandSolder, symbol Device:R
- removed R26, R27: 5.1kΩ, Resistor_SMD:R_0603_1608Metric_Pad0.98x0.95mm_HandSolder, symbol Device:R
- removed R28, R32: 1kΩ, Resistor_SMD:R_0603_1608Metric_Pad0.98x0.95mm_HandSolder, symbol Device:R
- removed R29, R30: 0Ω, Resistor_SMD:R_0805_2012Metric_Pad1.20x1.40mm_HandSolder, symbol Device:R
- removed R31: 1kΩ, Resistor_SMD:R_1206_3216Metric_Pad1.30x1.75mm_HandSolder, symbol Device:R
- removed SW1: USB | PS, Connector_PinHeader_2.54mm:PinHeader_1x03_P2.54mm_Vertical, symbol Switch:SW_SPDT
- removed SW4, SW5: Switch, Button_Switch_SMD:SW_SPST_SKQG_WithStem, symbol Switch:SW_Push
- removed U1: LD1117AV33, Package_TO_SOT_THT:TO-220-3_Vertical, symbol Regulator_Linear:LD1117S33TR_SOT223
- removed U5: CP2102N-A01-GQFN28, Package_DFN_QFN:QFN-28-1EP_5x5mm_P0.5mm_EP3.35x3.35mm, symbol Interface_USB:CP2102N-Axx-xQFN28
- removed U8: ESP32-WROOM-32D, RF_Module:ESP32-WROOM-32D, symbol RF_Module:ESP32-WROOM-32D
- added C14, C15, C16, C17: 10uF, Capacitor_THT:CP_Radial_D6.3mm_P2.50mm, symbol Device:C_Polarized_Small
- added J10: Rotary Encoder, Connector_JST:JST_EH_B4B-EH-A_1x04_P2.50mm_Vertical, symbol Connector:Conn_01x04_Socket
- added J11, J3, J9: Conn_01x08_Socket, Connector_PinSocket_2.54mm:PinSocket_1x08_P2.54mm_Vertical, symbol Connector:Conn_01x08_Socket
- added Q3: IRL520, Package_TO_SOT_THT:TO-220-3_Vertical, symbol Transistor_FET:IRL6283M
- added R21, R22, R35, R52, R53: 10k, Resistor_THT:R_Axial_DIN0207_L6.3mm_D2.5mm_P7.62mm_Horizontal, symbol Device:R
- added RN1, RN2: R_Network08, Resistor_THT:R_Array_SIP9, symbol Device:R_Network08
- added U10: ULN2803A, Package_DIP:DIP-18_W7.62mm_LongPads, symbol Transistor_Array:ULN2803A
- added U11: ESP32-DevKitC, Esp:ESP32-DevKitC, symbol Esp:ESP32-DevKitC
- added U4: 74HC595, Package_DIP:DIP-16_W7.62mm_Socket_LongPads, symbol 74xx:74HC595
- R1, R10, R11, R12, R13, R14, R15, R16, R2, R3, R4, R5, R6, R7, R8, R9: footprint (none) -> Resistor_THT:R_Axial_DIN0207_L6.3mm_D2.5mm_P7.62mm_Horizontal
- R19, R20: footprint Resistor_SMD:R_0603_1608Metric_Pad0.98x0.95mm_HandSolder -> Resistor_THT:R_Axial_DIN0207_L6.3mm_D2.5mm_P7.62mm_Horizontal
Connections:
- net +3.3V: now also U2.10 (~{SRCLR}), U7.10 (~{SRCLR}), C14.1, C15.1, C16.1, C17.1, R21.1, R22.1, R35.1, R53.1, RN1.1 (common), RN2.1 (common), U11.1 (3V3), U4.10 (~{SRCLR}), U4.16 (VCC)
- net +5V: now also U10.10 (COM)
- net GND: now also C14.2, C15.2, C16.2, C17.2, J10.4 (Pin_4), Q3.3 (S), R52.2, U10.9 (GND), U11.38 (GND), U4.8 (GND)
- net at R4.1: now also U6.5 (GPB4), RN2.5 (R4); no longer U6.4 (GPB3)
- net at R4.2: now also J11.4 (Pin_4)
- net Chan16: now reaches U9.1 (I1)
- net Chan16: now also U7.7 (QH)
- net Chan15: now reaches U9.2 (I2)
- net Chan15: now also U7.6 (QG)
- net Chan14: now reaches U9.3 (I3)
- net Chan14: now also U7.5 (QF)
- net Chan13: now reaches U9.4 (I4)
- net Chan13: now also U7.4 (QE)
- net Chan12: now reaches U9.5 (I5)
- net Chan12: now also U7.3 (QD)
- net Chan11: now reaches U9.6 (I6)
- net Chan11: now also U7.2 (QC)
- net Chan10: now reaches U9.7 (I7)
- net Chan10: now also U7.1 (QB)
- net Chan9: now reaches U9.8 (I8)
- net Chan9: now also U7.15 (QA)
- net at R5.1: now also U6.4 (GPB3), RN2.6 (R5); no longer U6.5 (GPB4)
- net at R5.2: now also J11.5 (Pin_5)
- net at R6.1: now also U6.3 (GPB2), RN2.7 (R6); no longer U6.6 (GPB5)
- net at R6.2: now also J11.6 (Pin_6)
- net at U6.1 (GPB0): now also R8.1, RN2.9 (R8); no longer R1.1
- net at R20.2, U6.12 (SCK): now also U11.11 (ADC2_CH7/GPIO27)
- net at R19.2, U6.13 (SDA): now also U11.10 (DAC_2/ADC2_CH9/GPIO26)
- net at U6.2 (GPB1): now also R7.1, RN2.8 (R7); no longer R2.1
- net at U6.21 (GPA0): now also R16.1, RN1.9 (R8); no longer R9.1
- net at U6.22 (GPA1): now also R15.1, RN1.8 (R7); no longer R10.1
- net at U6.23 (GPA2): now also R14.1, RN1.7 (R6); no longer R11.1
- net at U6.24 (GPA3): now also R13.1, RN1.6 (R5); no longer R12.1
- net at U6.25 (GPA4): now also R12.1, RN1.5 (R4); no longer R13.1
- net at U6.26 (GPA5): now also R11.1, RN1.4 (R3); no longer R14.1
- net at U6.27 (GPA6): now also R10.1, RN1.3 (R2); no longer R15.1
- net at U6.28 (GPA7): now also R9.1, RN1.2 (R1); no longer R16.1
- net at R3.1: now also U6.6 (GPB5), RN2.4 (R3); no longer U6.3 (GPB2)
- net at U6.7 (GPB6): now also R2.1, RN2.3 (R2); no longer R7.1
- net at U6.8 (GPB7): now also R1.1, RN2.2 (R1); no longer R8.1
- net at R3.2: now also J11.3 (Pin_3)
- net at R13.2: now also J3.5 (Pin_5)
- net at R11.2: now also J3.3 (Pin_3)
- net at R9.2: now also J3.1 (Pin_1)
- net at R1.2: now also J11.1 (Pin_1)
- net at R7.2: now also J11.7 (Pin_7)
- net at R14.2: now also J3.6 (Pin_6)
- net at U2.11 (SRCLK), U7.11 (SRCLK): now also U11.36 (GPIO22), U4.11 (SRCLK)
- net at U2.12 (RCLK), U7.12 (RCLK): now also U11.33 (GPIO21), U4.12 (RCLK)
- net at U2.13 (~{OE}), U7.13 (~{OE}): now also Q3.1 (D), R53.2, U4.13 (~{OE})
- net at U2.14 (SER): now also U11.31 (GPIO19)
- net at R10.2: now also J3.2 (Pin_2)
- net at R12.2: now also J3.4 (Pin_4)
- net at R15.2: now also J3.7 (Pin_7)
- net at R16.2: now also J3.8 (Pin_8)
- net at R2.2: now also J11.2 (Pin_2)
- net at R8.2: now also J11.8 (Pin_8)
- net at U7.9 (QH'): now also U4.14 (SER)
- net 1 renamed Chan1
- net 2 renamed Chan2
- net 3 renamed Chan3
- net 4 renamed Chan4
- net 5 renamed Chan5
- net 6 renamed Chan6
- net 7 renamed Chan7
- net 8 renamed Chan8
- new net: J10.1 (Pin_1), R35.2, U11.9 (DAC_1/ADC2_CH8/GPIO25)
- new net: Q3.2 (G), R52.1, U11.37 (GPIO23)
- new net: J10.2 (Pin_2), R22.2, U11.8 (32K_XN/GPIO33/ADC1_CH5)
- new net: J10.3 (Pin_3), R21.2, U11.7 (32K_XP/GPIO32/ADC1_CH4)
- new net: J9.1 (Pin_1), U10.18 (O1)
- new net: J9.2 (Pin_2), U10.17 (O2)
- new net: J9.3 (Pin_3), U10.16 (O3)
- new net: J9.4 (Pin_4), U10.15 (O4)
- new net: J9.5 (Pin_5), U10.14 (O5)
- new net: J9.6 (Pin_6), U10.13 (O6)
- new net: J9.7 (Pin_7), U10.12 (O7)
- new net: J9.8 (Pin_8), U10.11 (O8)
- new net Chan17: U10.8 (I8), U4.15 (QA)
- new net Chan18: U10.7 (I7), U4.1 (QB)
- new net Chan19: U10.6 (I6), U4.2 (QC)
- new net Chan20: U10.5 (I5), U4.3 (QD)
- new net Chan21: U10.4 (I4), U4.4 (QE)
- new net Chan22: U10.3 (I3), U4.5 (QF)
- new net Chan23: U10.2 (I2), U4.6 (QG)
- new net Chan24: U10.1 (I1), U4.7 (QH)
- no-connect marks 41 -> 26
Other:
- note removed: "Power Supply"
- note removed: "Programming Circuit"
- note removed: "UsbToSerial"
- moved on the sheet: J2, J4, R1, R10, R11, R12, R13, R14, R15, R16, R19, R2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
